File: PowerMeter_EADOG.brd (EAGLE design)
At the start: 74 x 32 mm, 49 parts, among them J1 PSS 254/4W, J2 PSS 254/4W, Q2 PDTC114YT, Q3 8MHz, U1 SN75176BD, U2 SN75176BD, U3 IP4220CZ6,125, U4 XC6206P332MR, U5 ATXMEGA32A4U

Commit message: - adding SD-Card option - moving push button to the center
Parts:
- added C8, C9: 4u7, rcl:C0603
- added R3, R7: 4k7, rcl:R0603
- added U6: MICROSD_SPI_MODE, con-molex-microsd:MICRO_SD_CONNECTOR
- R10: value 10k -> 4k7
- moved S1 2.77 mm to (68.2, 12.5)
Connections:
- removed net CSB_LCD: LCD1.38, R10.2, U5.20
- removed net D6_SCK: LCD1.29, U5.21
- removed net D7_MOSI: LCD1.28, U5.23
- removed net N$11: U5.28
- removed net N$14: U5.22
- new net CSB: LCD1.38, R10.2, R3.1, U5.20, U6.2
- new net MISO: R7.1, U5.22, U6.7
- new net MOSI: LCD1.28, U5.23, U6.3
- new net SCK: LCD1.29, U5.21, U6.5
- new net SW_SD: U5.28, U6.SW2
- net +3V3: now also C8.1, C9.1, R3.2, R7.2, U6.4
- net GND: now also C8.2, C9.2, U6.6, U6.SW1
Routing:
- net MOSI: track 0.00 -> 69.6 mm, vias 0 -> 2
- net CSB: track 0.00 -> 67.3 mm, vias 0 -> 3
- net SCK: track 0.00 -> 50.6 mm, vias 0 -> 2
- net CSB_LCD: track 46.8 -> 0.00 mm, vias 2 -> 0
- net LCD_DIM: track 66.8 -> 107.7 mm
- net MISO: track 0.00 -> 22.1 mm, vias 0 -> 1
- net D6_SCK: track 21.3 -> 0.00 mm, vias 1 -> 0
- net SW_SD: track 0.00 -> 21.1 mm, vias 0 -> 1
- net D7_MOSI: track 19.1 -> 0.00 mm, vias 1 -> 0
- net +3V3: track 149.4 -> 164.3 mm, vias 6 -> 7
- net GND: track 43.7 -> 37.7 mm, vias 37 -> 47
- net USER_SW: track 26.0 -> 27.8 mm
- net +5V: track 149.4 -> 149.2 mm, vias 2 -> 4
Other:
- board text added: "Place Display or SD-Card"
- board text added: "v1.1"
