File: PowerMeter_EADOG.sch (EAGLE design)
At the start: 49 parts, among them J1 PSS 254/4W, J2 PSS 254/4W, Q2 PDTC114YT, Q3 8MHz, U1 SN75176BD, U2 SN75176BD, U3 IP4220CZ6,125, U4 XC6206P332MR, U5 ATXMEGA32A4U

Commit message: - adding SD-Card option - moving push button to the center
Parts:
- added C8, C9: 4u7, rcl:C-EUC0603
- added R3, R7: 4k7, rcl:R-EU_R0603
- added U6: MICROSD_SPI_MODE, con-molex-microsd:MICROSD_SPI_MODE
- R10: value 10k -> 4k7
Connections:
- removed net CSB_LCD: LCD1.38_CSB, R10.2, U5.PD0
- removed net D6_SCK: LCD1.29_D6, U5.PD1
- removed net D7_MOSI: LCD1.28_D7, U5.PD3
- removed net N$11: U5.PE0
- removed net N$14: U5.PD2
- new net CSB: LCD1.38_CSB, R10.2, R3.1, U5.PD0, U6./CS
- new net MISO: R7.1, U5.PD2, U6.DO
- new net MOSI: LCD1.28_D7, U5.PD3, U6.DI
- new net SCK: LCD1.29_D6, U5.PD1, U6.CLK
- new net SW_SD: U5.PE0, U6.SW2
- net +3V3: now also C8.1, C9.1, R3.2, R7.2, U6.VDD
- net GND: now also C8.2, C9.2, U6.SW1, U6.VSS
Other:
- note added: "Place µSD-Card OR Display"
- note added: "v1.1"
- note removed: "v1.0"
- moved on the sheet: C1, C2, C6, Q2, R1, R10, R2, R5, S1
